Commit message: Edited URDF and lidar.xacro

File: src/joe_cart/description/lidar.xacro (robot description, xacro)
@@ -4,5 +4,5 @@
         <parent link="chassis"/>
         <child link="laser_frame"/>
-        <origin xyz="0.1 0 0.175" rpy="0 0 0"/>
+        <origin xyz="0.1 0 0.4" rpy="0 0 0"/>
     </joint>
     <link name="laser_frame">
@@ -10,5 +10,5 @@
             <origin xyz="0 0 0"/>
             <geometry>
-                <cylinder length="0.1" radius="0.05"/>
+                <cylinder length="0.08" radius="0.05"/>
             </geometry>
             <material name="red"/>

File: src/joe_cart/description/robot.urdf.xacro (robot description, xacro)
@@ -3,5 +3,4 @@
     <xacro:include filename="robot_core.xacro" />
     <xacro:include filename="ros2_control.xacro"/>
-    <!-- <xacro:include filename="gazebo_control.xacro" /> -->
     <xacro:include filename="lidar.xacro"/>
 </robot>

File: src/joe_cart/description/robot_core.xacro (robot description, xacro)
@@ -36,18 +36,18 @@
     <link name="chassis">
         <visual>
-            <origin xyz="0.15 0 0.075"/>
+            <origin xyz="0.18 0 0.2"/>
             <geometry>
-                <box size="0.3 0.3 0.15"/>
+                <box size="0.36 0.36 0.4"/>
             </geometry>
             <material name="white"/>
         </visual>
         <collision>
-            <origin xyz="0.15 0 0.075"/>
+            <origin xyz="0.18 0 0.2"/>
             <geometry>
-                <box size="0.3 0.3 0.15"/>
+                <box size="0.36 0.36 0.4"/>
             </geometry>
         </collision>
-        <xacro:inertial_box mass="0.5" x="0.3" y="0.3" z="0.15">
-            <origin xyz="0.15 0 0.075" rpy="0 0 0"/>
+        <xacro:inertial_box mass="0.5" x="0.36" y="0.36" z="0.4">
+            <origin xyz="0.18 0 0.2" rpy="0 0 0"/>
         </xacro:inertial_box>
     </link>
@@ -59,5 +59,5 @@
         <parent link="base_link"/>
         <child link="left_wheel"/>
-        <origin xyz="0 0.175 0" rpy="-${pi/2} 0 0" />
+        <origin xyz="0 0.2 0" rpy="-${pi/2} 0 0" />
         <axis xyz="0 0 1"/>
     </joint>
@@ -85,5 +85,5 @@
         <parent link="base_link"/>
         <child link="right_wheel"/>
-        <origin xyz="0 -0.175 0" rpy="${pi/2} 0 0" />
+        <origin xyz="0 -0.2 0" rpy="${pi/2} 0 0" />
         <axis xyz="0 0 -1"/>
     </joint>

File: src/joe_cart/description/ros2_control.xacro (robot description, xacro)
@@ -32,5 +32,5 @@
             <param name="baud_rate">57600</param>
             <param name="timeout">1000</param>
-            <param name="enc_counts_per_rev">830</param>
+            <param name="enc_counts_per_rev">3440</param>
         </hardware>
         <joint name="left_wheel_joint">

Commit message: Some Changes

File: src/joe_cart/description/lidar.xacro (robot description, xacro)
@@ -4,5 +4,5 @@
         <parent link="chassis"/>
         <child link="laser_frame"/>
-        <origin xyz="0.1 0 0.175" rpy="0 0 0"/>
+        <origin xyz="0.1 0 0.3" rpy="0 0 0"/>
     </joint>
     <link name="laser_frame">
@@ -10,5 +10,5 @@
             <origin xyz="0 0 0"/>
             <geometry>
-                <cylinder length="0.1" radius="0.05"/>
+                <cylinder length="0.08" radius="0.05"/>
             </geometry>
             <material name="red"/>

File: src/joe_cart/description/robot_core.xacro (robot description, xacro)
@@ -29,5 +29,5 @@
     </link>
     <!-- CHASSIS LINK -->
-    <joint name="chassis_joint" type="fixed">
+     <joint name="chassis_joint" type="fixed">
         <parent link="base_link"/>
         <child link="chassis"/>
@@ -36,7 +36,7 @@
     <link name="chassis">
         <visual>
-            <origin xyz="0.15 0 0.075"/>
+            <origin xyz="0.18 0 0.2"/>
             <geometry>
-                <box size="0.3 0.3 0.15"/>
+                <box size="0.36 0.36 0.4"/>
             </geometry>
             <material name="white"/>
@@ -45,9 +45,9 @@
             <origin xyz="0.15 0 0.075"/>
             <geometry>
-                <box size="0.3 0.3 0.15"/>
+                <box size="0.36 0.36 0.4"/>
             </geometry>
         </collision>
-        <xacro:inertial_box mass="0.5" x="0.3" y="0.3" z="0.15">
-            <origin xyz="0.15 0 0.075" rpy="0 0 0"/>
+        <xacro:inertial_box mass="0.5" x="0.36" y="0.36" z="0.4">
+            <origin xyz="0.18 0 0.2" rpy="0 0 0"/>
         </xacro:inertial_box>
     </link>

File: src/joe_cart/description/ros2_control.xacro (robot description, xacro)
@@ -29,5 +29,5 @@
             <param name="right_wheel_name">right_wheel_joint</param>
             <param name="loop_rate">30</param>
-            <param name="device">/dev/ttyACM0</param>
+            <param name="device">/dev/ttyUSB0</param>
             <param name="baud_rate">57600</param>
             <param name="timeout">1000</param>
