Commit message: Edited URDF,PID values and new map

File: src/joe_cart/description/robot_core.xacro (robot description, xacro)
@@ -32,5 +32,5 @@
         <parent link="base_link"/>
         <child link="chassis"/>
-        <origin xyz="-0.1 0 0"/>
+        <origin xyz="-0.1 0 0" rpy="0 0 ${pi}"/>
     </joint>
     <link name="chassis">
@@ -43,10 +43,10 @@
         </visual>
         <collision>
-            <origin xyz="0.15 0 0.075"/>
+            <origin xyz="0.18 0 0.2"/>
             <geometry>
                 <box size="0.36 0.36 0.4"/>
             </geometry>
         </collision>
-        <xacro:inertial_box mass="0.5" x="0.36" y="0.36" z="0.4">
+        <xacro:inertial_box mass="6.5" x="0.36" y="0.36" z="0.4">
             <origin xyz="0.18 0 0.2" rpy="0 0 0"/>
         </xacro:inertial_box>
@@ -59,5 +59,5 @@
         <parent link="base_link"/>
         <child link="left_wheel"/>
-        <origin xyz="0 0.175 0" rpy="-${pi/2} 0 0" />
+        <origin xyz="-0.1 0.2 0" rpy="-${pi/2} 0 0" />
         <axis xyz="0 0 1"/>
     </joint>
@@ -65,5 +65,5 @@
         <visual>
             <geometry>
-                <cylinder radius="0.05" length="0.04"/>
+                <cylinder radius="0.0325" length="0.025"/>
             </geometry>
             <material name="blue"/>
@@ -71,9 +71,9 @@
         <collision>
             <geometry>
-                <cylinder radius="0.05" length="0.04"/>
+                <cylinder radius="0.0325" length="0.025"/>
             </geometry>
         </collision>
-        <xacro:inertial_cylinder mass="0.1" length="0.04" radius="0.05">
-            <origin xyz="0 0 0" rpy="0 0 0"/>
+        <xacro:inertial_cylinder mass="0.1" length="0.025" radius="0.0325">
+            <origin xyz="-0.1 0 0" rpy="0 0 0"/>
         </xacro:inertial_cylinder>
     </link>
@@ -85,5 +85,5 @@
         <parent link="base_link"/>
         <child link="right_wheel"/>
-        <origin xyz="0 -0.175 0" rpy="${pi/2} 0 0" />
+        <origin xyz="-0.1 -0.2 0" rpy="${pi/2} 0 0" />
         <axis xyz="0 0 -1"/>
     </joint>
@@ -91,5 +91,5 @@
         <visual>
             <geometry>
-                <cylinder radius="0.05" length="0.04"/>
+                <cylinder radius="0.0325" length="0.025"/>
             </geometry>
             <material name="blue"/>
@@ -97,9 +97,9 @@
         <collision>
             <geometry>
-                <cylinder radius="0.05" length="0.04"/>
+                <cylinder radius="0.0325" length="0.025"/>
             </geometry>
         </collision>
-        <xacro:inertial_cylinder mass="0.1" length="0.04" radius="0.05">
-            <origin xyz="0 0 0" rpy="0 0 0"/>
+        <xacro:inertial_cylinder mass="0.1" length="0.025" radius="0.0325">
+            <origin xyz="-0.1 0 0" rpy="0 0 0"/>
         </xacro:inertial_cylinder>
     </link>
@@ -116,5 +116,5 @@
         <visual>
             <geometry>
-                <sphere radius="0.05"/>
+                <sphere radius="0.0325"/>
             </geometry>
             <material name="black"/>
@@ -122,8 +122,8 @@
         <collision>
             <geometry>
-                <sphere radius="0.05"/>
+                <sphere radius="0.0325"/>
             </geometry>
         </collision>
-        <xacro:inertial_sphere mass="0.1" radius="0.05">
+        <xacro:inertial_sphere mass="0.1" radius="0.0325">
             <origin xyz="0 0 0" rpy="0 0 0"/>
         </xacro:inertial_sphere>

File: src/joe_cart/description/ros2_control.xacro (robot description, xacro)
@@ -33,6 +33,6 @@
             <param name="timeout">1000</param>
             <param name="enc_counts_per_rev">830</param>
-            <param name="enc_cpr_left_motor">830</param>
-            <param name="enc_cpr_right_motor">830</param>
+            <param name="enc_cpr_left_motor">825</param>
+            <param name="enc_cpr_right_motor">825</param>
         </hardware>
         <joint name="left_wheel_joint">

Commit message: Added a better map

File: src/joe_cart/description/robot_core.xacro (robot description, xacro)
@@ -60,5 +60,5 @@
         <child link="left_wheel"/>
         <origin xyz="-0.1 0.2 0" rpy="-${pi/2} 0 0" />
-        <axis xyz="0 0 1"/>
+        <axis xyz="0 0 -1"/>
     </joint>
     <link name="left_wheel">
@@ -86,5 +86,5 @@
         <child link="right_wheel"/>
         <origin xyz="-0.1 -0.2 0" rpy="${pi/2} 0 0" />
-        <axis xyz="0 0 -1"/>
+        <axis xyz="0 0 1"/>
     </joint>
     <link name="right_wheel">

Commit message: Added Navigation waypoint file

File: src/joe_cart/description/robot_core.xacro (robot description, xacro)
@@ -60,5 +60,5 @@
         <child link="left_wheel"/>
         <origin xyz="-0.1 0.2 0" rpy="-${pi/2} 0 0" />
-        <axis xyz="0 0 -1"/>
+        <axis xyz="0 0 1"/>
     </joint>
     <link name="left_wheel">

File: src/joe_cart/description/ros2_control.xacro (robot description, xacro)
@@ -29,5 +29,5 @@
             <param name="right_wheel_name">right_wheel_joint</param>
             <param name="loop_rate">30</param>
-            <param name="device">/dev/ttyUSB0</param>
+            <param name="device">/dev/ttyACM1</param>
             <param name="baud_rate">57600</param>
             <param name="timeout">1000</param>

Commit message: Sprinting

File: src/joe_cart/description/robot_core.xacro (robot description, xacro)
@@ -17,4 +17,7 @@
         <color rgba="1 0 0 1"/>
     </material>
+    <!-- Define common properties -->
+    <xacro:property name="wheel_radius" value="0.0285" />
+    <xacro:property name="wheel_separation" value="0.44" />
     <!-- BASE LINK -->
     <link name="base_link">
@@ -28,109 +31,69 @@
     <link name="base_footprint">
     </link>
-    <!-- CHASSIS LINK -->
-     <joint name="chassis_joint" type="fixed">
+    <!-- CHASSIS LINK (corresponds to base_link in NEW file) -->
+    <joint name="chassis_joint" type="fixed">
         <parent link="base_link"/>
         <child link="chassis"/>
-        <origin xyz="-0.1 0 0" rpy="0 0 ${pi}"/>
+        <origin xyz="0 0 0" rpy="0 0 ${pi}"/>
     </joint>
     <link name="chassis">
+        <inertial>
+            <origin xyz="-0.0124711888668452 4.68604114422927E-05 0.269752234729229" rpy="0 0 0" />
+            <mass value="7.40564073717936" />
+            <inertia ixx="0.0840963831782375" ixy="1.14103457957399E-07" ixz="-6.77908469162018E-07"
+                     iyy="0.0690566081420881" iyz="5.11060740929003E-08" izz="0.114286230084613" />
+        </inertial>
         <visual>
-            <origin xyz="0.18 0 0.2"/>
+            <origin xyz="0 0 0" rpy="0 0 0" />
             <geometry>
-                <box size="0.36 0.36 0.4"/>
+                <mesh filename="package://joe_cart/meshes/base_link.STL" />
             </geometry>
             <material name="white"/>
         </visual>
         <collision>
-            <origin xyz="0.18 0 0.2"/>
+            <origin xyz="0 0 0" rpy="0 0 0" />
             <geometry>
-                <box size="0.36 0.36 0.4"/>
+                <mesh filename="package://joe_cart/meshes/base_link.STL" />
             </geometry>
         </collision>
-        <xacro:inertial_box mass="6.5" x="0.36" y="0.36" z="0.4">
-            <origin xyz="0.18 0 0.2" rpy="0 0 0"/>
-        </xacro:inertial_box>
     </link>
     <gazebo reference="chassis">
         <material>Gazebo/White</material>
     </gazebo>
-    <!-- LEFT WHEEL LINK -->
-    <joint name="left_wheel_joint" type="continuous">
-        <parent link="base_link"/>
-        <child link="left_wheel"/>
-        <origin xyz="-0.1 0.2 0" rpy="-${pi/2} 0 0" />
-        <axis xyz="0 0 1"/>
-    </joint>
-    <link name="left_wheel">
-        <visual>
-            <geometry>
-                <cylinder radius="0.0325" length="0.025"/>
-            </geometry>
-            <material name="blue"/>
-        </visual>
-        <collision>
-            <geometry>
-                <cylinder radius="0.0325" length="0.025"/>
-            </geometry>
-        </collision>
-        <xacro:inertial_cylinder mass="0.1" length="0.025" radius="0.0325">
-            <origin xyz="-0.1 0 0" rpy="0 0 0"/>
-        </xacro:inertial_cylinder>
-    </link>
-    <gazebo reference="left_wheel">
-        <material>Gazebo/Blue</material>
-    </gazebo>
-    <!-- RIGHT WHEEL LINK -->
-    <joint name="right_wheel_joint" type="continuous">
-        <parent link="base_link"/>
-        <child link="right_wheel"/>
-        <origin xyz="-0.1 -0.2 0" rpy="${pi/2} 0 0" />
-        <axis xyz="0 0 1"/>
-    </joint>
-    <link name="right_wheel">
-        <visual>
-            <geometry>
-                <cylinder radius="0.0325" length="0.025"/>
-            </geometry>
-            <material name="blue"/>
-        </visual>
-        <collision>
-            <geometry>
-                <cylinder radius="0.0325" length="0.025"/>
-            </geometry>
-        </collision>
-        <xacro:inertial_cylinder mass="0.1" length="0.025" radius="0.0325">
-            <origin xyz="-0.1 0 0" rpy="0 0 0"/>
-        </xacro:inertial_cylinder>
-    </link>
-    <gazebo reference="right_wheel">
-        <material>Gazebo/Blue</material>
-    </gazebo>
-    <!-- CASTER WHEEL LINK -->
-    <joint name="caster_wheel_joint" type="fixed">
-        <parent link="chassis"/>
-        <child link="caster_wheel"/>
-        <origin xyz="0.24 0 0"/>
-    </joint>
-    <link name="caster_wheel">
-        <visual>
-            <geometry>
-                <sphere radius="0.0325"/>
-            </geometry>
-            <material name="black"/>
-        </visual>
-        <collision>
-            <geometry>
-                <sphere radius="0.0325"/>
-            </geometry>
-        </collision>
-        <xacro:inertial_sphere mass="0.1" radius="0.0325">
-            <origin xyz="0 0 0" rpy="0 0 0"/>
-        </xacro:inertial_sphere>
-    </link>
-    <gazebo reference="caster_wheel">
-        <material>Gazebo/Black</material>
-        <mu1 value="0.001"/>
-        <mu2 value="0.001"/>
-    </gazebo>
+    <!-- Wheel Macro -->
+    <xacro:macro name="wheel" params="prefix reflect">
+        <link name="${prefix}_wheel">
+            <inertial>
+                <origin xyz="${reflect * 4.1702E-10} ${reflect * 0.003762} -1.1536E-09" rpy="0 0 0" />
+                <mass value="0.028216" />
+                <inertia ixx="1.1938E-05" ixy="${-reflect * 8.1598E-14}" ixz="${reflect * 8.2976E-15}"
+                         iyy="2.2184E-05" iyz="${reflect * 3.2808E-13}" izz="1.1939E-05" />
+            </inertial>
+            <visual>
+                <origin xyz="0 0 0" rpy="0 0 0" />
+                <geometry>
+                    <mesh filename="package://joe_cart/meshes/${prefix}_wheel.STL" />
+                </geometry>
+                <material name="blue"/>
+            </visual>
+            <collision>
+                <origin xyz="0 0 0" rpy="0 0 0" />
+                <geometry>
+                    <mesh filename="package://joe_cart/meshes/${prefix}_wheel.STL" />
+                </geometry>
+            </collision>
+        </link>
+        <joint name="${prefix}_wheel_joint" type="continuous">
+            <origin xyz="0.1615 ${reflect * wheel_separation/2} ${-wheel_radius}" rpy="0 0 0" />
+            <parent link="base_link" />
+            <child link="${prefix}_wheel" />
+            <axis xyz="0 1 0" />
+        </joint>
+        <gazebo reference="${prefix}_wheel">
+            <material>Gazebo/Blue</material>
+        </gazebo>
+    </xacro:macro>
+    <!-- Use the wheel macro -->
+    <xacro:wheel prefix="right" reflect="-1" />
+    <xacro:wheel prefix="left" reflect="1" />
 </robot>

Commit message: URDF fixes

File: src/joe_cart/description/robot_core.xacro (robot description, xacro)
@@ -85,5 +85,5 @@
         </link>
         <joint name="${prefix}_wheel_joint" type="continuous">
-            <origin xyz="0.1615 ${reflect * wheel_separation/2} ${-wheel_radius}" rpy="0 0 0" />
+            <origin xyz="-0.1615 ${reflect * wheel_separation/2} ${-wheel_radius}" rpy="0 0 0" />
             <parent link="base_link" />
             <child link="${prefix}_wheel" />

Commit message: Updated rviz

File: src/joe_cart/description/robot_core.xacro (robot description, xacro)
@@ -16,4 +16,7 @@
     <material name="red">
         <color rgba="1 0 0 1"/>
+    </material>
+    <material name="green">
+        <color rgba="0 1 0 1" />
     </material>
     <!-- BASE LINK -->
@@ -40,5 +43,5 @@
                 <box size="0.36 0.36 0.4"/>
             </geometry>
-            <material name="white"/>
+            <material name="green"/>
         </visual>
         <collision>
